File: hat.brd (EAGLE design)
At the start: 65 x 56 mm, 3 parts, among them K1 PIN20X2

Commit message: WS2812B board
Parts:
- removed USE_REG: (no value), jumper:JP1
- added C1, C2, C3: 0.1uF, SparkFun:0603-CAP
- added D3: Green, Testing:0603-LED-ALT1
- added L1, L10, L11, L12, L13, L14, L15, L16, L17, L18, L19, L2, L20, L21, L22, L23, L24, L25, L26, L27, L28, L29, L3, L30, L31, L32, L33, L34, L35, L36, L37, L38, L39, L4, L40, L41, L42, L43, L44, L45, L46, L47, L48, L5, L6, L7, L8, L9: WS2812B, adafruit:WS2812B
- added Q1: 8/16/20MHz, Testing:RESONATOR-SMD-1:1
- added R2: 10K, SparkFun:0603-RES
- added R6: 330, SparkFun:0603-RES
- added S1: Reset, Testing:TACTILE-SWITCH-SMD-ALT01
- added SJ1: JUMPER-PAD-2-NC_BY_TRACE, SparkFun-Passives:PAD-JUMPER-2-NC_BY_TRACE_YES_SILK
- added SV1: (no value), con-lstb:MA06-1
- added U1: ATMEGA328, SparkFun:TQFP32-08
- moved U$1 16.8 mm to (23.7, 1.43)
Connections:
- new net A0: U1.23
- new net A1: U1.24
- new net A2: U1.25
- new net A3: U1.26
- new net A6: U1.19
- new net A7: U1.22
- new net AREF: C1.2, U1.20
- new net D10: L1.4-DIN, U1.14
- new net D2: U1.32
- new net D3: U1.1
- new net D4: U1.2
- new net D5: U1.9
- new net D6: U1.10
- new net D7: U1.11
- new net D8: U1.12
- new net D9: U1.13
- new net DTR: C2.2
- new net MISO: U1.16
- new net MOSI: U1.15
- new net N$1: L10.4-DIN, L9.2-DOUT
- new net N$10: L11.2-DOUT, L12.4-DIN
- new net N$11: L12.2-DOUT, L13.4-DIN
- new net N$12: L13.2-DOUT, L14.4-DIN
- new net N$13: L14.2-DOUT, L15.4-DIN
- new net N$14: L15.2-DOUT, L16.4-DIN
- new net N$15: L17.2-DOUT, L18.4-DIN
- new net N$17: L19.2-DOUT, L20.4-DIN
- new net N$18: L20.2-DOUT, L21.4-DIN
- new net N$19: L21.2-DOUT, L22.4-DIN
- new net N$2: L1.2-DOUT, L2.4-DIN
- new net N$20: L22.2-DOUT, L23.4-DIN
- new net N$21: L23.2-DOUT, L24.4-DIN
- new net N$22: L25.2-DOUT, L26.4-DIN
- new net N$23: L26.2-DOUT, L27.4-DIN
- new net N$24: L27.2-DOUT, L28.4-DIN
- new net N$25: L28.2-DOUT, L29.4-DIN
- new net N$26: L29.2-DOUT, L30.4-DIN
- new net N$27: L30.2-DOUT, L31.4-DIN
- new net N$28: L31.2-DOUT, L32.4-DIN
- new net N$29: D3.A, R6.2
- new net N$3: L2.2-DOUT, L3.4-DIN
- new net N$30: Q1.3, U1.8
- new net N$31: Q1.1, U1.7
- new net N$32: L33.2-DOUT, L34.4-DIN
- new net N$33: L34.2-DOUT, L35.4-DIN
- new net N$34: L35.2-DOUT, L36.4-DIN
- new net N$35: L36.2-DOUT, L37.4-DIN
- new net N$36: L37.2-DOUT, L38.4-DIN
- new net N$37: L38.2-DOUT, L39.4-DIN
- new net N$38: L39.2-DOUT, L40.4-DIN
- new net N$39: L41.2-DOUT, L42.4-DIN
- new net N$4: L3.2-DOUT, L4.4-DIN
- new net N$40: L42.2-DOUT, L43.4-DIN
- new net N$41: L43.2-DOUT, L44.4-DIN
- new net N$42: L44.2-DOUT, L45.4-DIN
- new net N$43: L45.2-DOUT, L46.4-DIN
- new net N$44: L46.2-DOUT, L47.4-DIN
- new net N$45: L47.2-DOUT, L48.4-DIN
- new net N$46: L8.2-DOUT, L9.4-DIN
- new net N$47: L16.2-DOUT, L17.4-DIN
- new net N$48: L24.2-DOUT, L25.4-DIN
- new net N$49: L40.2-DOUT, L41.4-DIN
- new net N$5: L4.2-DOUT, L5.4-DIN
- new net N$50: L32.2-DOUT, L33.4-DIN
- new net N$51: R6.1, SJ1.2
- new net N$6: L5.2-DOUT, L6.4-DIN
- new net N$7: L6.2-DOUT, L7.4-DIN
- new net N$8: L7.2-DOUT, L8.4-DIN
- new net N$9: L10.2-DOUT, L11.4-DIN
- new net RESET: C2.1, R2.1, S1.3, S1.4, U1.29
- new net RXI: U1.30
- new net SCK: SJ1.1, U1.17
- new net TXO: U1.31
- net +5V: now also C3.2, K1.2, K1.4, L1.1-VDD, L10.1-VDD, L11.1-VDD, L12.1-VDD, L13.1-VDD, L14.1-VDD, L15.1-VDD, L16.1-VDD, L17.1-VDD, L18.1-VDD, L19.1-VDD, L2.1-VDD, L20.1-VDD, L21.1-VDD, L22.1-VDD, L23.1-VDD, L24.1-VDD, L25.1-VDD, L26.1-VDD, L27.1-VDD, L28.1-VDD, L29.1-VDD, L3.1-VDD, L30.1-VDD, L31.1-VDD, L32.1-VDD, L33.1-VDD, L34.1-VDD, L35.1-VDD, L36.1-VDD, L37.1-VDD, L38.1-VDD, L39.1-VDD, L4.1-VDD, L40.1-VDD, L41.1-VDD, L42.1-VDD, L43.1-VDD, L44.1-VDD, L45.1-VDD, L46.1-VDD, L47.1-VDD, L48.1-VDD, L5.1-VDD, L6.1-VDD, L7.1-VDD, L8.1-VDD, L9.1-VDD, R2.2, U1.18, U1.4, U1.6; no longer USE_REG.1
- net GND: now also C1.1, C3.1, D3.C, L1.3-GND, L10.3-GND, L11.3-GND, L12.3-GND, L13.3-GND, L14.3-GND, L15.3-GND, L16.3-GND, L17.3-GND, L18.3-GND, L19.3-GND, L2.3-GND, L20.3-GND, L21.3-GND, L22.3-GND, L23.3-GND, L24.3-GND, L25.3-GND, L26.3-GND, L27.3-GND, L28.3-GND, L29.3-GND, L3.3-GND, L30.3-GND, L31.3-GND, L32.3-GND, L33.3-GND, L34.3-GND, L35.3-GND, L36.3-GND, L37.3-GND, L38.3-GND, L39.3-GND, L4.3-GND, L40.3-GND, L41.3-GND, L42.3-GND, L43.3-GND, L44.3-GND, L45.3-GND, L46.3-GND, L47.3-GND, L48.3-GND, L5.3-GND, L6.3-GND, L7.3-GND, L8.3-GND, L9.3-GND, Q1.2, S1.1, S1.2, U1.21, U1.3, U1.5
- net I2C_SCL: now also U1.28
- net I2C_SDA: now also U1.27
- net N$16: now also L18.2-DOUT, L19.4-DIN; no longer K1.2, K1.4, USE_REG.2
Routing:
- net +5V: track 0.00 -> 476.2 mm, vias 0 -> 1
- net RESET: track 0.00 -> 122.8 mm, vias 0 -> 1
- net SCK: track 0.00 -> 118.3 mm, vias 0 -> 1
- net N$50: track 0.00 -> 74.5 mm
- net N$48: track 0.00 -> 74.3 mm
- net N$47: track 0.00 -> 74.3 mm
- net N$49: track 0.00 -> 74.3 mm
- net N$46: track 0.00 -> 74.3 mm
- net D10: track 0.00 -> 18.3 mm, vias 0 -> 1
- net N$16: track 17.2 -> 4.43 mm
- net N$9: track 0.00 -> 4.43 mm
- net N$14: track 0.00 -> 4.43 mm
- net N$13: track 0.00 -> 4.43 mm
- net N$12: track 0.00 -> 4.43 mm
- net N$11: track 0.00 -> 4.43 mm
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