File: hat.sch (EAGLE design)
At the start: 2 parts, among them K1 PIN20X2

Commit message: WS2812B board
Parts:
- removed USE_REG: (no value), jumper:JP1E
- added C1, C2, C3: 0.1uF, SparkFun:CAP0603-CAP
- added D3: Green, Testing:LED
- added L1, L10, L11, L12, L13, L14, L15, L16, L17, L18, L19, L2, L20, L21, L22, L23, L24, L25, L26, L27, L28, L29, L3, L30, L31, L32, L33, L34, L35, L36, L37, L38, L39, L4, L40, L41, L42, L43, L44, L45, L46, L47, L48, L5, L6, L7, L8, L9: WS2812B, adafruit:WS2812B
- added Q1: 8/16/20MHz, Testing:RESONATOR1:1
- added R2: 10K, SparkFun:RESISTOR0603-RES
- added R6: 330, SparkFun:RESISTOR0603-RES
- added S1: Reset, Testing:SWITCH-MOMENTARY-2SMD-ALT01
- added SJ1: JUMPER-PAD-2-NC_BY_TRACE, SparkFun-Passives:JUMPER-PAD-2-NC_BY_TRACE
- added SV1: (no value), con-lstb:MA06-1
- added U1: ATMEGA328, SparkFun:ATMEGA168
Connections:
- new net A0: U1.PC0(ADC0)
- new net A1: U1.PC1(ADC1)
- new net A2: U1.PC2(ADC2)
- new net A3: U1.PC3(ADC3)
- new net A6: U1.ADC6
- new net A7: U1.ADC7
- new net AREF: C1.2, U1.AREF
- new net D10: L1.DIN, U1.PB2(SS/OC1B)
- new net D2: U1.PD2(INT0)
- new net D3: U1.PD3(INT1)
- new net D4: U1.PD4(XCK/T0)
- new net D5: U1.PD5(T1)
- new net D6: U1.PD6(AIN0)
- new net D7: U1.PD7(AIN1)
- new net D8: U1.PB0(ICP)
- new net D9: U1.PB1(OC1A)
- new net DTR: C2.2
- new net MISO: U1.PB4(MISO)
- new net MOSI: U1.PB3(MOSI/OC2)
- new net N$1: L10.DIN, L9.DOUT
- new net N$10: L11.DOUT, L12.DIN
- new net N$11: L12.DOUT, L13.DIN
- new net N$12: L13.DOUT, L14.DIN
- new net N$13: L14.DOUT, L15.DIN
- new net N$14: L15.DOUT, L16.DIN
- new net N$15: L17.DOUT, L18.DIN
- new net N$17: L19.DOUT, L20.DIN
- new net N$18: L20.DOUT, L21.DIN
- new net N$19: L21.DOUT, L22.DIN
- new net N$2: L1.DOUT, L2.DIN
- new net N$20: L22.DOUT, L23.DIN
- new net N$21: L23.DOUT, L24.DIN
- new net N$22: L25.DOUT, L26.DIN
- new net N$23: L26.DOUT, L27.DIN
- new net N$24: L27.DOUT, L28.DIN
- new net N$25: L28.DOUT, L29.DIN
- new net N$26: L29.DOUT, L30.DIN
- new net N$27: L30.DOUT, L31.DIN
- new net N$28: L31.DOUT, L32.DIN
- new net N$29: D3.A, R6.2
- new net N$3: L2.DOUT, L3.DIN
- new net N$30: Q1.3, U1.PB7(XTAL2/TOSC2)
- new net N$31: Q1.1, U1.PB6(XTAL1/TOSC1)
- new net N$32: L33.DOUT, L34.DIN
- new net N$33: L34.DOUT, L35.DIN
- new net N$34: L35.DOUT, L36.DIN
- new net N$35: L36.DOUT, L37.DIN
- new net N$36: L37.DOUT, L38.DIN
- new net N$37: L38.DOUT, L39.DIN
- new net N$38: L39.DOUT, L40.DIN
- new net N$39: L41.DOUT, L42.DIN
- new net N$4: L3.DOUT, L4.DIN
- new net N$40: L42.DOUT, L43.DIN
- new net N$41: L43.DOUT, L44.DIN
- new net N$42: L44.DOUT, L45.DIN
- new net N$43: L45.DOUT, L46.DIN
- new net N$44: L46.DOUT, L47.DIN
- new net N$45: L47.DOUT, L48.DIN
- new net N$46: L8.DOUT, L9.DIN
- new net N$47: L16.DOUT, L17.DIN
- new net N$48: L24.DOUT, L25.DIN
- new net N$49: L40.DOUT, L41.DIN
- new net N$5: L4.DOUT, L5.DIN
- new net N$50: L32.DOUT, L33.DIN
- new net N$51: R6.1, SJ1.2
- new net N$6: L5.DOUT, L6.DIN
- new net N$7: L6.DOUT, L7.DIN
- new net N$8: L7.DOUT, L8.DIN
- new net N$9: L10.DOUT, L11.DIN
- new net RESET: C2.1, R2.1, S1.2, U1.PC6(/RESET)
- new net RXI: U1.PD0(RXD)
- new net SCK: SJ1.1, U1.PB5(SCK)
- new net TXO: U1.PD1(TXD)
- net +5V: now also C3.2, K1.2, K1.4, L1.VDD, L10.VDD, L11.VDD, L12.VDD, L13.VDD, L14.VDD, L15.VDD, L16.VDD, L17.VDD, L18.VDD, L19.VDD, L2.VDD, L20.VDD, L21.VDD, L22.VDD, L23.VDD, L24.VDD, L25.VDD, L26.VDD, L27.VDD, L28.VDD, L29.VDD, L3.VDD, L30.VDD, L31.VDD, L32.VDD, L33.VDD, L34.VDD, L35.VDD, L36.VDD, L37.VDD, L38.VDD, L39.VDD, L4.VDD, L40.VDD, L41.VDD, L42.VDD, L43.VDD, L44.VDD, L45.VDD, L46.VDD, L47.VDD, L48.VDD, L5.VDD, L6.VDD, L7.VDD, L8.VDD, L9.VDD, R2.2, U1.AVCC, U1.VCC@1, U1.VCC@2; no longer USE_REG.1
- net GND: now also C1.1, C3.1, D3.C, L1.GND, L10.GND, L11.GND, L12.GND, L13.GND, L14.GND, L15.GND, L16.GND, L17.GND, L18.GND, L19.GND, L2.GND, L20.GND, L21.GND, L22.GND, L23.GND, L24.GND, L25.GND, L26.GND, L27.GND, L28.GND, L29.GND, L3.GND, L30.GND, L31.GND, L32.GND, L33.GND, L34.GND, L35.GND, L36.GND, L37.GND, L38.GND, L39.GND, L4.GND, L40.GND, L41.GND, L42.GND, L43.GND, L44.GND, L45.GND, L46.GND, L47.GND, L48.GND, L5.GND, L6.GND, L7.GND, L8.GND, L9.GND, Q1.2, S1.1, U1.AGND, U1.GND@1, U1.GND@2
- net I2C_SCL: now also U1.PC5(ADC5/SCL)
- net I2C_SDA: now also U1.PC4(ADC4/SDA)
- net N$16: now also L18.DOUT, L19.DIN; no longer K1.2, K1.4, USE_REG.2
