File: ws2812-hat.brd (EAGLE design)
At the start: 65 x 56 mm, 61 parts, among them K1 PIN20X2, Q1 8/16/20MHz, U1 ATMEGA328

Commit message: More finished-er
Parts:
- removed C1: 0.1uF, SparkFun:0603-CAP
- removed SV1: (no value), con-lstb:MA06-1
- added C4: 0.1uf, rcl:C0805K
- added JP1: FTDI Basic, SparkFun:1X06
- moved U$1 16.4 mm to (7.30, 0.95)
- moved Q1 0.16 mm to (19.8, 40.5)
- moved U1 0.16 mm to (12.9, 43.0)
Connections:
- net +5V: now also JP1.4
- net AREF: now also C4.1; no longer C1.2
- net DTR: now also JP1.1
- net GND: now also C4.2, JP1.5, JP1.6; no longer C1.1
- net RXI: now also JP1.3
- net TXO: now also JP1.2
Routing:
- net RXI: track 0.00 -> 57.1 mm
- net TXO: track 0.00 -> 56.3 mm
- net +5V: track 476.2 -> 513.0 mm
- net DTR: track 0.00 -> 28.0 mm
- net RESET: track 122.8 -> 126.9 mm
- net AREF: track 0.00 -> 1.67 mm
- net D10: track 18.3 -> 19.9 mm
