File: ws2812-hat.sch (EAGLE design)
At the start: 60 parts, among them K1 PIN20X2, Q1 8/16/20MHz, U1 ATMEGA328

Commit message: More finished-er
Parts:
- removed C1: 0.1uF, SparkFun:CAP0603-CAP
- removed SV1: (no value), con-lstb:MA06-1
- added C4: 0.1uf, rcl:C-EUC0805K
- added JP1: FTDI Basic, SparkFun:ARDUINO_SERIAL_PROGRAMPTH
Connections:
- net +5V: now also JP1.VCC
- net AREF: now also C4.1; no longer C1.2
- net DTR: now also JP1.DTR
- net GND: now also C4.2, JP1.CTS, JP1.GND; no longer C1.1
- net RXI: now also JP1.TXO
- net TXO: now also JP1.RXI
Changed lines of the file:
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@@
 <part name="P+2" library="supply1" deviceset="+5V" device=""/>
 <part name="GND4" library="supply1" deviceset="GND" device=""/>
-<part name="SV1" library="con-lstb" deviceset="MA06-1" device=""/>
-<part name="P+4" library="supply1" deviceset="+5V" device=""/>
-<part name="GND1" library="supply1" deviceset="GND" device=""/>
 <part name="L9" library="adafruit" deviceset="WS2812B" device=""/>
 <part name="L10" library="adafruit" deviceset="WS2812B" device=""/>
@@
 <part name="C3" library="SparkFun" deviceset="CAP" device="0603-CAP" value="0.1uF"/>
 <part name="GND8" library="SparkFun" deviceset="GND" device=""/>
-<part name="C1" library="SparkFun" deviceset="CAP" device="0603-CAP" value="0.1uF"/>
 <part name="GND9" library="SparkFun" deviceset="GND" device=""/>
 <part name="R6" library="SparkFun" deviceset="RESISTOR" device="0603-RES" value="330"/>
@@
 <part name="P+10" library="supply1" deviceset="+5V" device=""/>
 <part name="P+11" library="supply1" deviceset="+5V" device=""/>
+<part name="JP1" library="SparkFun" deviceset="ARDUINO_SERIAL_PROGRAM" device="PTH" value="FTDI Basic"/>
+<part name="P+4" library="supply1" deviceset="+5V" device=""/>
+<part name="GND1" library="supply1" deviceset="GND" device=""/>
+<part name="C4" library="rcl" deviceset="C-EU" device="C0805K" value="0.1uf"/>
 </parts>
 <sheets>
@@
 <instance part="P+2" gate="1" x="162.56" y="175.26"/>
 <instance part="GND4" gate="1" x="162.56" y="149.86"/>
-<instance part="SV1" gate="1" x="83.82" y="152.4" rot="MR180"/>
-<instance part="P+4" gate="1" x="106.68" y="167.64" smashed="yes">
-<attribute name="VALUE" x="109.22" y="170.18" size="1.778" layer="96" rot="R180"/>
-</instance>
-<instance part="GND1" gate="1" x="106.68" y="142.24"/>
 <instance part="L9" gate="G$1" x="162.56" y="134.62"/>
 <instance part="L10" gate="G$1" x="175.26" y="134.62"/>
@@
 </instance>
 <instance part="GND8" gate="1" x="347.98" y="68.58"/>
-<instance part="C1" gate="G$1" x="342.9" y="109.22" smashed="yes" rot="R180">
-<attribute name="NAME" x="343.916" y="109.347" size="1.778" layer="95"/>
-<attribute name="VALUE" x="343.916" y="104.521" size="1.778" layer="96"/>
-</instance>
 <instance part="GND9" gate="1" x="342.9" y="99.06"/>
 <instance part="R6" gate="G$1" x="391.16" y="50.8"/>
@@
 <instance part="P+10" gate="1" x="335.28" y="147.32"/>
 <instance part="P+11" gate="1" x="347.98" y="86.36"/>
+<instance part="JP1" gate="G$1" x="88.9" y="165.1"/>
+<instance part="P+4" gate="1" x="106.68" y="177.8"/>
+<instance part="GND1" gate="1" x="104.14" y="154.94"/>
+<instance part="C4" gate="G$1" x="342.9" y="109.22"/>
 </instances>
 <busses>
@@
 </segment>
 <segment>
-<pinref part="GND1" gate="1" pin="GND"/>
-<wire x1="106.68" y1="154.94" x2="106.68" y2="144.78" width="0.1524" layer="91"/>
-</segment>
-<segment>
 <pinref part="L16" gate="G$1" pin="GND"/>
 <wire x1="251.46" y1="129.54" x2="251.46" y2="127" width="0.1524" layer="91"/>
@@
 <segment>
 <wire x1="342.9" y1="101.6" x2="342.9" y2="104.14" width="0.1524" layer="91"/>
-<pinref part="C1" gate="G$1" pin="1"/>
 <pinref part="GND9" gate="1" pin="GND"/>
+<pinref part="C4" gate="G$1" pin="2"/>
 </segment>
 <segment>
@@
 <junction x="226.06" y="12.7"/>
 </segment>
+<segment>
+<pinref part="JP1" gate="G$1" pin="GND"/>
+<pinref part="GND1" gate="1" pin="GND"/>
+<wire x1="93.98" y1="172.72" x2="104.14" y2="172.72" width="0.1524" layer="91"/>
+<wire x1="104.14" y1="172.72" x2="104.14" y2="170.18" width="0.1524" layer="91"/>
+<pinref part="JP1" gate="G$1" pin="CTS"/>
+<wire x1="104.14" y1="170.18" x2="104.14" y2="157.48" width="0.1524" layer="91"/>
+<wire x1="93.98" y1="170.18" x2="104.14" y2="170.18" width="0.1524" layer="91"/>
+<junction x="104.14" y="170.18"/>
+</segment>
 </net>
 <net name="+3V3" class="0">
@@
 </segment>
 <segment>
-<pinref part="P+4" gate="1" pin="+5V"/>
-<wire x1="106.68" y1="157.48" x2="106.68" y2="165.1" width="0.1524" layer="91"/>
-</segment>
-<segment>
 <pinref part="K1" gate="G$1" pin="2"/>
 <wire x1="58.42" y1="170.18" x2="63.5" y2="170.18" width="0.1524" layer="91"/>
@@
 <pinref part="P+11" gate="1" pin="+5V"/>
 </segment>
+<segment>
+<pinref part="P+4" gate="1" pin="+5V"/>
+<wire x1="106.68" y1="175.26" x2="106.68" y2="167.64" width="0.1524" layer="91"/>
+<pinref part="JP1" gate="G$1" pin="VCC"/>
+<wire x1="106.68" y1="167.64" x2="93.98" y2="167.64" width="0.1524" layer="91"/>
+</segment>
 </net>
 <net name="ID_SCL" class="0">
@@
 <wire x1="342.9" y1="114.3" x2="342.9" y2="111.76" width="0.1524" layer="91"/>
 <label x="350.52" y="114.3" size="1.778" layer="95"/>
-<pinref part="C1" gate="G$1" pin="2"/>
 <pinref part="U1" gate="G$1" pin="AREF"/>
+<pinref part="C4" gate="G$1" pin="1"/>
 </segment>
 </net>
@@
 <label x="411.48" y="104.14" size="1.27" layer="95" xref="yes"/>
 </segment>
+<segment>
+<wire x1="93.98" y1="162.56" x2="96.52" y2="162.56" width="0.1524" layer="91"/>
+<pinref part="JP1" gate="G$1" pin="RXI"/>
+<label x="96.52" y="162.56" size="1.27" layer="95" xref="yes"/>
+</segment>
 </net>
 <net name="D9" class="0">
@@
 <label x="320.04" y="129.54" size="1.27" layer="95" rot="R180" xref="yes"/>
 </segment>
+<segment>
+<wire x1="93.98" y1="160.02" x2="96.52" y2="160.02" width="0.1524" layer="91"/>
+<pinref part="JP1" gate="G$1" pin="DTR"/>
+<label x="96.52" y="160.02" size="1.27" layer="95" xref="yes"/>
+</segment>
 </net>
 <net name="RXI" class="0">
@@
 <label x="411.48" y="106.68" size="1.27" layer="95" xref="yes"/>
 </segment>
-</net>
+<segment>
+<wire x1="93.98" y1="165.1" x2="96.52" y2="165.1" width="0.1524" layer="91"/>
+<pinref part="JP1" gate="G$1" pin="TXO"/>
+<label x="96.52" y="165.1" size="1.27" layer="95" xref="yes"/>
+</segment>
+</net>
